File: board/board.kicad_pcb (KiCad board)
At the start: 2 copper layers, 21 x 13 mm, 1 part

Commit message: initial
Parts:
- added C1: 47uF, Capacitor_SMD:C_1210_3225Metric, F.Cu at (146.8, 92.6)
- added C2: 47uF, Capacitor_SMD:C_1210_3225Metric, F.Cu at (146.8, 97.4)
- added C3: 10uF, Capacitor_SMD:C_0603_1608Metric, F.Cu at (157.2, 99.1)
- added C4: 1uF, Capacitor_SMD:C_0603_1608Metric, F.Cu at (164.5, 101.4)
- added C5: 100nF, Capacitor_SMD:C_0603_1608Metric, F.Cu at (163.0, 101.4)
- added C6: 47nF, Capacitor_SMD:C_0603_1608Metric, B.Cu at (174.4, 91.9)
- added D1: MMSZ5230BT1G, Diode_SMD:D_SOD-123, F.Cu at (158.2, 91.4)
- added FB1: BLM18RK221SN1D, Capacitor_SMD:C_0603_1608Metric, F.Cu at (157.2, 100.6)
- added J1: 003_power, on_edge:on_edge_2x05_device, F.Cu at (140.0, 96.5)
- added J2: Conn_01x02_Male, Connector_PinHeader_2.54mm:PinHeader_1x02_P2.54mm_Vertical, F.Cu at (168.4, 94.5)
- added J3: 022_battery_cells, on_edge:on_edge_2x05_host, F.Cu at (185.0, 96.5)
- added Q1: Q_PNP_BCEC, Package_TO_SOT_SMD:TO-252-3_TabPin4, F.Cu at (152.2, 95.8)
- added Q2: Q_PNP_BCEC, Package_TO_SOT_SMD:TO-252-3_TabPin4, F.Cu at (174.5, 95.7)
- added R1: 91R, Resistor_SMD:R_0603_1608Metric, F.Cu at (149.1, 102.2)
- added R10: 0.25R, Resistor_SMD:R_1206_3216Metric, B.Cu at (176.4, 92.7)
- added R2: 270R, Resistor_SMD:R_0603_1608Metric, F.Cu at (152.2, 102.2)
- added R3: 75k, Resistor_SMD:R_0603_1608Metric, F.Cu at (160.0, 101.4)
- added R4: 100k, Resistor_SMD:R_0603_1608Metric, F.Cu at (161.5, 101.4)
- added R5: 10k, Resistor_SMD:R_0603_1608Metric, F.Cu at (167.2, 99.3)
- added R6: 10k, Resistor_SMD:R_0603_1608Metric, F.Cu at (174.5, 102.1)
- added R7: 100R, Resistor_SMD:R_0603_1608Metric, F.Cu at (171.5, 102.1)
- added R8: 10k, Resistor_SMD:R_0603_1608Metric, F.Cu at (168.8, 99.3)
- added R9: 0.25R, Resistor_SMD:R_1206_3216Metric, B.Cu at (178.7, 92.6)
- added TH1: NTCG103JF103FT1, Resistor_SMD:R_0402_1005Metric, F.Cu at (167.0, 101.8)
- added TH2: NTCG103JF103FT1, Resistor_SMD:R_0402_1005Metric, F.Cu at (169.2, 101.8)
- added U1: DS2711E+, Package_SO:TSSOP-16_4.4x3.6mm_P0.4mm, F.Cu at (163.3, 95.1)
- LOGO1: moved to B.Cu
- moved LOGO1 4.34 mm to (151.1, 94.8), turned to 180 degrees
Routing:
- net GND: track 0.00 -> 69.3 mm, vias 0 -> 6
- net /charger/In: track 0.00 -> 42.8 mm, vias 0 -> 3
- net Net-(D1-Pad1): track 0.00 -> 40.3 mm, vias 0 -> 2
- net /charger/BTH: track 0.00 -> 27.8 mm, vias 0 -> 2
- net /charger/BTM: track 0.00 -> 19.6 mm, vias 0 -> 2
- net Net-(R2-Pad2): track 0.00 -> 16.4 mm
- net Net-(R7-Pad1): track 0.00 -> 12.3 mm
- net Net-(C3-Pad1): track 0.00 -> 11.3 mm
- net /charger/BTL: track 0.00 -> 9.04 mm, vias 0 -> 1
- net /charger/LED2: track 0.00 -> 7.75 mm
- net Net-(R8-Pad1): track 0.00 -> 7.62 mm
- net Net-(C2-Pad2): track 0.00 -> 7.20 mm
- net /charger/LED1: track 0.00 -> 6.73 mm
- net Net-(R5-Pad1): track 0.00 -> 6.38 mm
- net Net-(D1-Pad2): track 0.00 -> 4.01 mm
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Other:
- board size 21 x 13 mm -> 45 x 13 mm
- board text added: "osf.003"
- board text added: "osf.022"
- board text added: "osf.b105.v0.1"
